File: SCH_PCB/IGN01A.kicad_pcb (KiCad board)
At the start: 2 copper layers, 50 x 45 mm, 25 parts, among them IC1 ATMEGA328-A, J1 PWR, J2 IGN, J3 HEADER_1x09, J5 ISP, Q1 IRF7413ZPBF, U1 MPL3115A2

Commit message: Minor PCB tweaks
Routing:
- net VDD: track 170.9 -> 173.2 mm
